Commit message: rvizでurdfが動作します

File: so100_description/so100.urdf (robot description, URDF)
Before this commit: robot so_arm100, 7 links, 6 joints
Links:
- link base: geometry collision mesh filename=package://kinematics_so100/so100_description/assets/Base.stl; visual mesh filename=package://kinematics_so100/so100_description/assets/Base.stl
- link gripper: geometry visual mesh filename=package://kinematics_so100/so100_description/assets/Fixed_J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; visual mesh filename=package://kinematics_so100/so100_description/assets/Fixed_J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
- link jaw: geometry visual mesh filename=package://kinematics_so100/so100_description/assets/Moving_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
- link lower_arm: geometry collision mesh filename=package://kinematics_so100/so100_description/assets/Lower_A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; visual mesh filename=package://kinematics_so100/so100_description/assets/Lower_A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
- link shoulder: geometry collision mesh filename=package://kinematics_so100/so100_description/assets/Rotatio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; visual mesh filename=package://kinematics_so100/so100_description/assets/Rotatio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
- link upper_arm: geometry collision mesh filename=package://kinematics_so100/so100_description/assets/Upper_A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; visual mesh filename=package://kinematics_so100/so100_description/assets/Upper_A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
- link wrist: geometry collision mesh filename=package://kinematics_so100/so100_description/assets/Wrist_P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; visual mesh filename=package://kinematics_so100/so100_description/assets/Wrist_P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
